Commit message: fix: Complete ROS 2 Jazzy migration audit and repair
- Update all CMakeLists.txt to cmake_minimum_required 3.16
- Remove invalid find_package calls for runtime-only dependencies
- Convert Gazebo Classic sensor plugins to native Harmonic SDF sensors
- Fix ros2_control hardware plugin (GazeboSimSystem -> GZSimSystem)
- Create Gazebo Harmonic SDF 1.9 world files (empty.sdf, mini_pupper_home.sdf)
- Add ros_gz_bridge for clock, LiDAR, and IMU topic bridging
- Update Nav2 params: recoveries_server -> behavior_server, fix plugin names
- Fix controller YAML: joint_states_controller -> joint_state_broadcaster
- Fix SLAM launch files: PathJoinSubstitution and argument passing
- Add proper rclpy.shutdown() to Python driver nodes
- Correct package.xml dependency types and add missing dependencies
- Update CI workflow for Jazzy rosdep skip keys and actions/checkout v4

Co-authored-by: Cursor <cursoragent@cursor.com>

File: mini_pupper_description/urdf/mini_pupper/mini_pupper_description.urdf.xacro (robot description, xacro)
@@ -1489,5 +1489,5 @@
   <ros2_control name="GazeboSystem" type="system">
     <hardware>
-      <plugin>gz_ros2_control/GazeboSimSystem</plugin>
+      <plugin>gz_ros2_control/GZSimSystem</plugin>
     </hardware>
     <joint name="base_lf1">
@@ -1728,14 +1728,13 @@
   </gazebo>
   <gazebo reference="lidar_link">
-    <material>Gazebo/FlatBlack</material>
-    <sensor type="ray" name="lidar">
+    <sensor type="gpu_lidar" name="lidar">
       <always_on>true</always_on>
-      <update_rate>30</update_rate>
-      <pose>0 0 0 0 0 0</pose>
-      <visualize>false</visualize>
-      <ray>
+      <update_rate>10</update_rate>
+      <topic>lidar/scan</topic>
+      <gz_frame_id>lidar_link</gz_frame_id>
+      <lidar>
         <scan>
           <horizontal>
-            <samples>1040</samples>
+            <samples>360</samples>
             <resolution>1</resolution>
             <min_angle>0</min_angle>
@@ -1744,6 +1743,6 @@
         </scan>
         <range>
-          <min>0.2</min>
-          <max>50.0</max>
+          <min>0.12</min>
+          <max>12.0</max>
           <resolution>0.01</resolution>
         </range>
@@ -1753,34 +1752,13 @@
           <stddev>0.004</stddev>
         </noise>
-      </ray>
-      <!-- Gazebo Harmonic plugin name - may need adjustment based on gz_ros2_bridge -->
-      <plugin name="gazebo_ros_lidar_controller" filename="libgz_ros_ray_sensor.so">
-        <ros>
-          <remapping>~/out:=/scan</remapping>
-        </ros>
-        <output_type>sensor_msgs/LaserScan</output_type>
-        <frame_name>lidar_link</frame_name>
-        <!--min_intensity>100.0</min_intensity-->
-      </plugin>
+      </lidar>
+      <visualize>false</visualize>
     </sensor>
   </gazebo>
   <gazebo>
-    <!-- Ground truth odometry plugin - verify compatibility with Gazebo Harmonic -->
-    <plugin filename="libgz_ros_p3d.so" name="p3d_base_controller">
-      <ros>
-          <remapping>odom:=odom/ground_truth</remapping>
-      </ros>
-      <body_name>base_link</body_name>
-      <frame_name>world</frame_name>
-      <update_rate>10.0</update_rate>
-      <xyz_offset>0 0 0</xyz_offset>
-      <rpy_offset>0 0 0</rpy_offset>
-      <gaussian_noise>0.01</gaussian_noise>
-    </plugin>
-  </gazebo>
-  <gazebo>
-    <!-- Gazebo Harmonic ROS 2 Control plugin - Updated for Jazzy -->
-    <plugin filename="libgz_ros2_control.so" name="gz_ros2_control">
+    <plugin filename="gz_ros2_control-system" name="gz_ros2_control::GazeboSimROS2ControlPlugin">
       <parameters>$(find mini_pupper_description)/config/ros_control/mini_pupper_controller.yaml</parameters>
+      <robot_param>robot_description</robot_param>
+      <robot_param_node>robot_state_publisher</robot_param_node>
     </plugin>
   </gazebo>
@@ -1797,18 +1775,22 @@
   </joint>
   <gazebo reference="imu_link">
-    <sensor name="imu_controller" type="imu">
+    <sensor name="imu_sensor" type="imu">
       <always_on>true</always_on>
-      <update_rate>50</update_rate>
-      <!-- IMU plugin - verify compatibility with Gazebo Harmonic -->
-      <plugin name="gazebo_ros_imu_sensor" filename="libgz_ros_imu_sensor.so">
-          <ros>
-              <namespace>/imu</namespace>
-              <remapping>~/out:=data</remapping>
-          </ros>
-      </plugin>
+      <update_rate>100</update_rate>
+      <topic>imu/data</topic>
+      <gz_frame_id>imu_link</gz_frame_id>
+      <imu>
+        <angular_velocity>
+          <x><noise type="gaussian"><mean>0.0</mean><stddev>2e-4</stddev></noise></x>
+          <y><noise type="gaussian"><mean>0.0</mean><stddev>2e-4</stddev></noise></y>
+          <z><noise type="gaussian"><mean>0.0</mean><stddev>2e-4</stddev></noise></z>
+        </angular_velocity>
+        <linear_acceleration>
+          <x><noise type="gaussian"><mean>0.0</mean><stddev>1.7e-2</stddev></noise></x>
+          <y><noise type="gaussian"><mean>0.0</mean><stddev>1.7e-2</stddev></noise></y>
+          <z><noise type="gaussian"><mean>0.0</mean><stddev>1.7e-2</stddev></noise></z>
+        </linear_acceleration>
+      </imu>
     </sensor>
   </gazebo>
-  <!--xacro:sensor_d435 parent="base_link">
-  <origin xyz="0.08 0.0 0.07" rpy="0 0 0" />
-  </xacro:sensor_d435-->
 </robot>

File: mini_pupper_description/urdf/mini_pupper_2/mini_pupper_description.urdf.xacro (robot description, xacro)
@@ -838,5 +838,5 @@
   <ros2_control name="GazeboSystem" type="system">
     <hardware>
-      <plugin>gz_ros2_control/GazeboSimSystem</plugin>
+      <plugin>gz_ros2_control/GZSimSystem</plugin>
     </hardware>
     <joint name="base_lf1">
@@ -1089,14 +1089,13 @@
   </gazebo>
   <gazebo reference="lidar_link">
-    <material>Gazebo/FlatBlack</material>
-    <sensor type="ray" name="lidar">
+    <sensor type="gpu_lidar" name="lidar">
       <always_on>true</always_on>
-      <update_rate>30</update_rate>
-      <pose>0 0 0 0 0 0</pose>
-      <visualize>false</visualize>
-      <ray>
+      <update_rate>10</update_rate>
+      <topic>lidar/scan</topic>
+      <gz_frame_id>lidar_link</gz_frame_id>
+      <lidar>
         <scan>
           <horizontal>
-            <samples>1040</samples>
+            <samples>360</samples>
             <resolution>1</resolution>
             <min_angle>0</min_angle>
@@ -1105,6 +1104,6 @@
         </scan>
         <range>
-          <min>0.2</min>
-          <max>50.0</max>
+          <min>0.12</min>
+          <max>12.0</max>
           <resolution>0.01</resolution>
         </range>
@@ -1114,33 +1113,13 @@
           <stddev>0.004</stddev>
         </noise>
-      </ray>
-      <!-- Gazebo Harmonic plugin name - may need adjustment based on gz_ros2_bridge -->
-      <plugin name="gazebo_ros_lidar_controller" filename="libgz_ros_ray_sensor.so">
-        <ros>
-          <remapping>~/out:=/scan</remapping>
-        </ros>
-        <output_type>sensor_msgs/LaserScan</output_type>
-        <frame_name>lidar_link</frame_name>
-      </plugin>
+      </lidar>
+      <visualize>false</visualize>
     </sensor>
   </gazebo>
   <gazebo>
-    <!-- Ground truth odometry plugin - verify compatibility with Gazebo Harmonic -->
-    <plugin filename="libgz_ros_p3d.so" name="p3d_base_controller">
-      <ros>
-        <remapping>odom:=odom/ground_truth</remapping>
-      </ros>
-      <body_name>base_link</body_name>
-      <frame_name>world</frame_name>
-      <update_rate>10.0</update_rate>
-      <xyz_offset>0 0 0</xyz_offset>
-      <rpy_offset>0 0 0</rpy_offset>
-      <gaussian_noise>0.01</gaussian_noise>
-    </plugin>
-  </gazebo>
-  <gazebo>
-    <!-- Gazebo Harmonic ROS 2 Control plugin - Updated for Jazzy -->
-    <plugin filename="libgz_ros2_control.so" name="gz_ros2_control">
+    <plugin filename="gz_ros2_control-system" name="gz_ros2_control::GazeboSimROS2ControlPlugin">
       <parameters>$(find mini_pupper_description)/config/ros_control/mini_pupper_2_controller.yaml</parameters>
+      <robot_param>robot_description</robot_param>
+      <robot_param_node>robot_state_publisher</robot_param_node>
     </plugin>
   </gazebo>
@@ -1157,14 +1136,21 @@
   </joint>
   <gazebo reference="imu_link">
-    <sensor name="imu_controller" type="imu">
+    <sensor name="imu_sensor" type="imu">
       <always_on>true</always_on>
-      <update_rate>50</update_rate>
-      <!-- IMU plugin - verify compatibility with Gazebo Harmonic -->
-      <plugin name="gazebo_ros_imu_sensor" filename="libgz_ros_imu_sensor.so">
-          <ros>
-              <namespace>/imu</namespace>
-              <remapping>~/out:=data</remapping>
-          </ros>
-      </plugin>
+      <update_rate>100</update_rate>
+      <topic>imu/data</topic>
+      <gz_frame_id>imu_link</gz_frame_id>
+      <imu>
+        <angular_velocity>
+          <x><noise type="gaussian"><mean>0.0</mean><stddev>2e-4</stddev></noise></x>
+          <y><noise type="gaussian"><mean>0.0</mean><stddev>2e-4</stddev></noise></y>
+          <z><noise type="gaussian"><mean>0.0</mean><stddev>2e-4</stddev></noise></z>
+        </angular_velocity>
+        <linear_acceleration>
+          <x><noise type="gaussian"><mean>0.0</mean><stddev>1.7e-2</stddev></noise></x>
+          <y><noise type="gaussian"><mean>0.0</mean><stddev>1.7e-2</stddev></noise></y>
+          <z><noise type="gaussian"><mean>0.0</mean><stddev>1.7e-2</stddev></noise></z>
+        </linear_acceleration>
+      </imu>
     </sensor>
   </gazebo>
@@ -1173,12 +1159,6 @@
     <visual>
       <geometry>
-        <box>
-          <size>0.02 0.02 0.02</size>
-        </box>
-      </geometry>
-      <material>
-        <ambient>0 0 1 1</ambient>
-        <diffuse>0 0 1 1</diffuse>
-      </material>
+        <box size="0.02 0.02 0.02"/>
+      </geometry>
     </visual>
   </link>
@@ -1191,6 +1171,7 @@
     <sensor type="camera" name="sim_camera">
       <always_on>true</always_on>
-      <update_rate>30.0</update_rate>
-      <visualize>true</visualize>
+      <update_rate>15.0</update_rate>
+      <topic>image_raw</topic>
+      <gz_frame_id>camera_link</gz_frame_id>
       <camera name="camera">
         <horizontal_fov>1.3962634</horizontal_fov>
@@ -1205,12 +1186,5 @@
         </clip>
       </camera>
-      <!-- Gazebo ROS plugin to publish /image_raw -->
-      <plugin name="camera_controller" filename="libgz_ros_camera.so">
-        <always_on>true</always_on>
-        <update_rate>30.0</update_rate>
-        <frame_name>camera_link</frame_name>
-        <image_topic_name>/image_raw</image_topic_name>
-        <!-- camera_info omitted to disable /camera_info -->
-      </plugin>
+      <visualize>true</visualize>
     </sensor>
   </gazebo>
